File: Eletronica/Esquemáticos/Segundo esquemático/Segundo esquemático.kicad_sch (KiCad schematic)
At the start: 31 parts, among them M1 Motor Esquerdo, M2 Motor Direito, Q1 BC547, Q2 BC547, SW1 Chave/Interruptor, SW2 Chave/Interruptor, U2 Medidor de Corrente ACS712, U3 Sensor 1 TCRT500, U4 Sensor 2 TCRT500, U5 Sensor 3 TCRT500, U6 Sensor 4 TCRT500

Commit message: Att
Adicionei algumas alterações locais ao git novo
Parts:
- R7, R8: value 560 -> 100
Connections:
- new net: U2.8 (VCC), U8. (Vcc), U9. (Vcc)
Changed lines of the file:
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@@
       (effects (font (size 1.27 1.27)))
     )
-    (property "Value" "560" (at 222.25 130.81 90)
+    (property "Value" "100" (at 222.25 130.81 90)
       (effects (font (size 1.27 1.27)))
     )
@@
       (effects (font (size 1.27 1.27)))
     )
-    (property "Value" "560" (at 223.52 96.52 90)
-      (effects (font (size 1.27 1.27)))
-    )
+    (property "Value" "100" (at 223.52 96.52 90)
+      (effects (font (size 1.27 1.27)))
+    )
